Commit message: Add robot arm configuration and update URDF for Krytn tray integration

File: src/bar_examples/krytn/robot_description/krytn.urdf.xacro (robot description, xacro)
@@ -11,4 +11,28 @@
     <origin xyz="0 0 0.15" rpy="0 0 0" />
   </xacro:lidar_2d>
+  <link name="krytn_tray">
+    <visual>
+      <!--Part/Body.-->
+      <origin rpy="0.0 -0.0 0.0" xyz="0.0 0.0 0.0"/>
+      <geometry>
+        <mesh filename="package://krytn_tray/meshes/krytn_tray_demo_00_Krytn_Tray.dae"/>
+      </geometry>
+    </visual>
+    <collision>
+      <!--Part/Body.-->
+      <origin rpy="0.0 -0.0 0.0" xyz="0.0 0.0 0.0"/>
+      <geometry>
+        <mesh filename="package://krytn_tray/meshes/krytn_tray_demo_00_Krytn_Tray.dae"/>
+      </geometry>
+    </collision>
+    <xacro:box_inertial_with_origin x="0.398" y="0.221" z="0.150" mass="1.0">
+      <origin xyz="0.0 0 0.00" rpy="0 0 0" />
+    </xacro:box_inertial_with_origin>
+  </link>
+  <joint name="tray_joint" type="fixed">
+    <parent link="base_link"/>
+    <child link="krytn_tray"/>
+    <origin rpy="0.0 -0.0 1.5707963267948966" xyz="-0.3 0.014 0.167"/>
+  </joint>
   <!-- Configure Control of Joints -->
   <ros2_control name="Krytn" type="system">

File: src/bar_examples/maci/robot_description/maci.urdf.xacro (robot description, xacro)
@@ -3,5 +3,5 @@
     <xacro:include filename="$(find magni_description)/urdf/inertial.xacro" />
     <xacro:include filename="$(find sensors)/realsense_d435/realsense.urdf.xacro" />
-    <!-- Include a UR10 -->
+    <!-- Include a UR5 -->
     <xacro:include filename="$(find ur_description)/urdf/ur_macro.xacro" />
     <xacro:arg name="ur_type" default="ur5e"/>

File: src/bar_examples/sensors/lidar_2d/lidar_2d.urdf.xacro (robot description, xacro)
@@ -37,7 +37,7 @@
                     </scan>
                     <range>
-                        <min>0.060</min>
-                        <max>5</max>
-                        <resolution>0.01</resolution>
+                        <min>0.060</min> <!-- minimum distance to detect -->
+                        <max>5</max> <!-- maximum distance to detect -->
+                        <resolution>0.01</resolution> <!-- resolution of the lidar, it can distinguish between 0.01m changes in distance -->
                     </range>
                     <noise>
