Commit message: Commits up till D 14

File: src/my_robot_arm/urdf/my_robot_arm.urdf (robot description, URDF)
Before this commit: robot my_robot_arm, 2 links, 1 joints
Joints:
- joint finger_joint: limit lower=0.0 upper=0.065 effort=1000.0 velocity=0.01 -> lower=-0.01 upper=0.078 effort=1000.0 velocity=1000.1; origin xyz=-0.0627 -0.00085 0.06 rpy=0.0 -0.0 0.0 -> xyz=-0.06 0.001 0.06 rpy=0.0 -0.0 0.0

File: src/my_robot_arm/urdf/my_robot_arm.urdf.xacro (robot description, xacro)
@@ -52,5 +52,5 @@
         <origin rpy="0.0 -0.0 0.0" xyz="-0.0627 -0.00085 0.06"/>
         <axis xyz="1 0 0"/>
-        <limit effort="1000.0" lower="0.0" upper="0.065" velocity="0.01"/>
+        <limit effort="1000.0" lower="0.0" upper="0.07" velocity="0.01"/>
     </joint>
     <joint name="gripper_joint" type="fixed">
@@ -62,5 +62,5 @@
             <plugin>gz_ros2_control/GazeboSimSystem</plugin>
         </hardware>
-        <joint name="finger_link">
+        <joint name="finger_joint">
             <command_interface name="position"/>
             <state_interface name="position">
